File: bobachest/bobachest.kicad_pcb (KiCad board)
At the start: 2 copper layers, 33 parts, among them Q1 PN2222A, Q2 PN2222A, Q3 PN2222A, Q4 PN2222A, Q5 PN2222A, U1 arduino_mini

Commit message: Bobachest update
Parts:
- added P1: CONN_01X02, Pin_Headers:Pin_Header_Straight_1x02, F.Cu at (152.4, 97.5)
- added REF**: MountingHole_2.2mm_M2, Mounting_Holes:MountingHole_2.2mm_M2, F.Cu at (84.8, 51.3)
- added REF**: MountingHole_2.2mm_M2, Mounting_Holes:MountingHole_2.2mm_M2, F.Cu at (84.8, 97.5)
- added REF**: MountingHole_2.2mm_M2, Mounting_Holes:MountingHole_2.2mm_M2, F.Cu at (170.2, 51.3)
- added REF**: MountingHole_2.2mm_M2, Mounting_Holes:MountingHole_2.2mm_M2, F.Cu at (170.2, 97.5)
- BAR1, BAR2: footprint Display:HDSP-48xx -> BarSegm:HDSP-48xx
- R1, R10, R11, R12, R13, R14, R15, R16, R17, R18, R2, R3, R4, R5, R6, R7, R8, R9: footprint Resistors_ThroughHole:Resistor_Horizontal_RM7mm -> Resistor7mm:Resistor_Horizontal_RM7mm
- RV1: footprint Potentiometers:Potentiometer_Bourns_3339H_Angular_ScrewUp -> Potentiometer_Trimmer-Suntan-TSR-3386P
- RV2: footprint Potentiometers:Potentiometer_Bourns_3339H_Angular_ScrewUp -> TRIMPOT:Potentiometer_Trimmer-Suntan-TSR-3386P
- moved RV1 48.1 mm to (140.2, 91.9)
- moved RV2 2.50 mm to (141.2, 57.4)
- moved R11 2.34 mm to (140.2, 85.4)
- moved R12 2.34 mm to (140.2, 64.1)
- moved R13 2.34 mm to (140.2, 70.2)
- moved R14 2.34 mm to (140.2, 76.3)
- moved R15 2.34 mm to (140.2, 82.4)
- moved R16 2.34 mm to (140.2, 79.3)
- moved R17 2.34 mm to (140.2, 73.2)
- moved R18 2.34 mm to (140.2, 67.1)
- moved U1 2.16 mm to (161.0, 72.8)
Connections:
- U1 pad 20: Net-(R18-Pad2) -> Net-(R12-Pad2)
- U1 pad 21: Net-(R17-Pad2) -> Net-(R18-Pad2)
- U1 pad 22: Net-(R16-Pad2) -> Net-(R13-Pad2)
- U1 pad 23: Net-(R15-Pad2) -> Net-(R17-Pad2)
- U1 pad 25: Net-(R13-Pad2) -> Net-(R16-Pad2)
- U1 pad 26: Net-(R12-Pad2) -> Net-(R15-Pad2)
- U1 pad 4: S4 -> S5
- U1 pad 5: S5 -> S4
Routing:
- net Net-(Q1-Pad1): track 0.00 -> 107.0 mm
- net B1: track 0.00 -> 80.5 mm
- net GND: track 0.00 -> 70.8 mm
- net B2: track 0.00 -> 69.1 mm
- net S1: track 0.00 -> 60.9 mm
- net B3: track 0.00 -> 57.8 mm
- net +9V: track 0.00 -> 53.5 mm
- net S4: track 0.00 -> 51.8 mm
- net S2: track 0.00 -> 51.3 mm
- net B4: track 0.00 -> 46.6 mm
- net S3: track 0.00 -> 41.8 mm
- net S5: track 0.00 -> 40.6 mm
- net B5: track 0.00 -> 35.3 mm
- net Net-(R12-Pad2): track 0.00 -> 6.52 mm
- net Net-(R18-Pad2): track 0.00 -> 6.31 mm
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Other:
- board outline added: 90.4 x 51.3 mm

Commit message: update
Other:
- net class Default: clearance 0.2 -> 0.1524
- rule trace_clearance: 0.2 -> 0.1524

Commit message: gerber files
Other:
- board text added: "Bobachest V1.0 - Designed by AngelLM www.angel-lm.com"
